File: PCB/WhimsyMatrix.sch (KiCad schematic (older format))
At the start: 96 parts, among them K1 KEYSW, K10 KEYSW, K11 KEYSW, K12 KEYSW, K13 KEYSW, K14 KEYSW, K15 KEYSW, K16 KEYSW, K17 KEYSW, K18 KEYSW, K19 KEYSW, K2 KEYSW, K20 KEYSW, K21 KEYSW, K22 KEYSW, K23 KEYSW, K24 KEYSW, K25 KEYSW, K26 KEYSW, K27 KEYSW, K28 KEYSW, K29 KEYSW, K3 KEYSW, K30 KEYSW, K31 KEYSW, K32 KEYSW, K33 KEYSW, K34 KEYSW, K35 KEYSW, K36 KEYSW, K37 KEYSW, K38 KEYSW, K39 KEYSW, K4 KEYSW, K40 KEYSW, K41 KEYSW, K42 KEYSW, K43 KEYSW, K44 KEYSW, K45 KEYSW, K46 KEYSW, K47 KEYSW, K5 KEYSW, K6 KEYSW, K7 KEYSW, K8 KEYSW, K9 KEYSW, SW1 Rotary_Encoder_Switch

Commit message: updated PCB design
Parts:
- K1, K10, K11, K12, K13, K14, K15, K16, K17, K18, K19, K21, K22, K23, K25, K26, K27, K29, K30, K31, K32, K33, K34, K35, K36, K37, K38, K39, K4, K40, K41, K42, K43, K44, K47, K5, K6, K7, K8, K9: footprint keebs:Mx_Alps_100 -> MX_Only:MXOnly-1U-NoLED
- K2, K20, K28, K46: footprint keebs:Mx_Alps_125 -> MX_Only:MXOnly-1.25U-NoLED
- K24: footprint keebs:Mx_Alps_200 -> MX_Only:MXOnly-2U-ReversedStabilizers-NoLED
- K3, K45: footprint keebs:Mx_Alps_150 -> MX_Only:MXOnly-1.5U-NoLED
- SW1: footprint SofleKeyboard-footprint:RotaryEncoder_Alps_EC11E-Switch_Vertical_H20mm-keebio_modified -> CustomPrints:RotaryEncoder_Alps_EC11E-Switch_Vertical_H20mm-keebio_modified
